File: Learning and desmistifyng KiCad first/YT/Prj 2 - Traffic light for Arduino/Prj 3 - Traffic light for Arduino.kicad_sch (KiCad schematic)
At the start: 11 parts, among them J2 Conn_01x04

Commit message: updates on demistifying kicad
Changed lines of the file:
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@@
 		(on_board yes)
 		(dnp no)
-		(fields_autoplaced yes)
 		(property "Reference" "R3"
-			(at 161.29 60.96 90)
+			(at 161.036 65.278 90)
 			(effects
 				(font
@@
 		)
 		(property "Value" "R"
-			(at 161.29 63.5 90)
+			(at 161.798 70.866 90)
 			(effects
 				(font
@@
 		(on_board yes)
 		(dnp no)
-		(fields_autoplaced yes)
 		(property "Reference" "D3"
-			(at 183.1975 59.69 0)
+			(at 181.356 64.77 0)
 			(effects
 				(font
@@
 		)
 		(property "Value" "LED"
-			(at 183.1975 62.23 0)
+			(at 181.356 70.358 0)
 			(effects
 				(font
@@
 		(on_board yes)
 		(dnp no)
-		(fields_autoplaced yes)
 		(property "Reference" "D2"
-			(at 183.1975 52.07 0)
+			(at 181.864 57.15 0)
 			(effects
 				(font
@@
 		)
 		(property "Value" "LED"
-			(at 183.1975 54.61 0)
+			(at 182.372 61.976 0)
 			(effects
 				(font
@@
 		(on_board yes)
 		(dnp no)
-		(fields_autoplaced yes)
 		(property "Reference" "R2"
-			(at 161.29 53.34 90)
+			(at 161.036 57.404 90)
 			(effects
 				(font
@@
 		)
 		(property "Value" "R"
-			(at 161.29 55.88 90)
+			(at 161.29 61.976 90)
 			(effects
 				(font
@@
 		(on_board yes)
 		(dnp no)
-		(fields_autoplaced yes)
 		(property "Reference" "D1"
-			(at 183.1975 44.45 0)
+			(at 181.61 49.53 0)
 			(effects
 				(font
@@
 		)
 		(property "Value" "LED"
-			(at 183.1975 46.99 0)
+			(at 181.356 54.356 0)
 			(effects
 				(font
@@
 		(on_board yes)
 		(dnp no)
-		(fields_autoplaced yes)
 		(property "Reference" "R1"
-			(at 161.29 45.72 90)
+			(at 161.544 49.784 90)
 			(effects
 				(font
@@
 		)
 		(property "Value" "R"
-			(at 161.29 48.26 90)
-			(effects
-				(font
+			(at 161.29 54.356 90)
+			(effects
+				(font
