File: Learning and desmistifyng KiCad first/YT/Prj 1 - DesignESP32 S 3/Prj 2 - DesignESP32 S 3.kicad_sch (KiCad schematic)
At the start: 0 parts

Commit message: updates
Other:
- title: (none) -> ESP32  sensor board-Root
Changed lines of the file:
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@@
 	(generator_version "9.0")
 	(paper "A4")
+	(title_block
+		(title "ESP32  sensor board-Root")
+	)
 	(sheet_instances
 		(path "/"
