File: Learning and desmistifyng KiCad first/KiCAD like a pro 1/PRJ 1 - LED TORCH/Prj 1 - LED  files/Prj 1 - LED Torch.kicad_pcb (KiCad board)
At the start: 2 copper layers, 88.5 x 25 mm, 5 parts, among them SW1 SW_DPST_x2

Commit message: add updates
Routing:
- net /LED_Cathode: track 82.0 -> 81.5 mm
Changed lines of the file:
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@@
 	)
 	(segment
-		(start 98.5 116)
-		(end 102.311 112.189)
+		(start 100.846534 113.653466)
+		(end 98.5 116)
 		(width 0.2)
 		(layer "F.Cu")
@@
 	)
 	(segment
-		(start 171.369 112.189)
+		(start 172.962792 113.782792)
 		(end 176.68 117.5)
 		(width 0.2)
@@
 	)
 	(segment
-		(start 102.311 112.189)
-		(end 171.369 112.189)
+		(start 169.115036 112.189)
+		(end 104.382068 112.189)
+		(width 0.2)
+		(layer "F.Cu")
+		(net 1)
+	)
+	(arc
+		(start 100.846534 113.653466)
+		(mid 102.468651 112.569602)
+		(end 104.382068 112.189)
+		(width 0.2)
+		(layer "F.Cu")
+		(net 1)
+	)
+	(arc
+		(start 172.962792 113.782792)
+		(mid 171.197426 112.603213)
+		(end 169.115036 112.189)
 		(width 0.2)
 		(layer "F.Cu")
@@
 	)
 	(segment
-		(start 125.162552 120.162552)
-		(end 144.657448 120.162552)
+		(start 125.807823 120.162552)
+		(end 142.774739 120.162552)
 		(width 0.2)
 		(layer "F.Cu")
@@
 	)
 	(segment
-		(start 144.657448 120.162552)
+		(start 145.988724 118.831276)
 		(end 147.32 117.5)
 		(width 0.2)
@@
 	)
 	(segment
-		(start 117.75 119.25)
-		(end 124.25 119.25)
+		(start 123.604728 119.25)
+		(end 117.75 119.25)
+		(width 0.2)
+		(layer "F.Cu")
+		(net 2)
+	)
+	(arc
+		(start 124.706276 119.706276)
+		(mid 125.21167 120.043969)
+		(end 125.807823 120.162552)
+		(width 0.2)
+		(layer "F.Cu")
+		(net 2)
+	)
+	(arc
+		(start 145.988724 118.831276)
+		(mid 144.514135 119.816564)
+		(end 142.774739 120.162552)
+		(width 0.2)
+		(layer "F.Cu")
+		(net 2)
+	)
+	(arc
+		(start 124.706276 119.706276)
+		(mid 124.200881 119.368582)
+		(end 123.604728 119.25)
 		(width 0.2)
 		(layer "F.Cu")
@@
 	)
 	(segment
-		(start 124.25 119.25)
-		(end 125.162552 120.162552)
-		(width 0.2)
-		(layer "F.Cu")
-		(net 2)
-	)
-	(segment
-		(start 105.5 113.19)
-		(end 103.85 113.19)
+		(start 104.675 113.19)
+		(end 105.5 113.19)
 		(width 0.2)
 		(layer "F.Cu")
@@
 	)
 	(segment
-		(start 103.85 113.19)
+		(start 103.266636 113.773363)
 		(end 98.5 118.54)
 		(width 0.2)
@@
 		(net 3)
 	)
+	(arc
+		(start 104.675 113.19)
+		(mid 103.912799 113.341611)
+		(end 103.266636 113.773363)
+		(width 0.2)
+		(layer "F.Cu")
+		(net 3)
+	)
 	(segment
-		(start 111.955418 120.81)
-		(end 117.75 115.015418)
+		(start 117.65616 115.109257)
+		(end 113.54921 119.216207)
 		(width 0.2)
 		(layer "F.Cu")
@@
 	)
 	(segment
-		(start 105.5 120.81)
-		(end 111.955418 120.81)
+		(start 109.701454 120.81)
+		(end 105.5 120.81)
 		(width 0.2)
 		(layer "F.Cu")
@@
 	)
 	(segment
-		(start 117.75 115.015418)
-		(end 117.75 114.75)
+		(start 117.882709 114.75)
+		(end 124.25 114.75)
 		(width 0.2)
 		(layer "F.Cu")
 		(net 4)
 	)
-	(segment
-		(start 117.75 114.75)
-		(end 124.25 114.75)
+	(arc
+		(start 113.54921 119.216207)
+		(mid 111.783844 120.395786)
+		(end 109.701454 120.81)
 		(width 0.2)
 		(layer "F.Cu")
+		(net 4)
+	)
+	(arc
+		(start 117.882709 114.75)
+		(mid 117.788869 114.788869)
+		(end 117.75 114.882709)
+		(width 0.2)
+		(layer "F.Cu")
+		(net 4)
+	)
+	(arc
+		(start 117.75 114.882709)
+		(mid 117.725611 115.005316)
+		(end 117.65616 115.109257)
+		(width 0.2)
+		(layer "F.Cu")
